File: board/board.kicad_pcb (KiCad board)
At the start: 2 copper layers, 50 x 81 mm, 59 parts, among them IC1 tps610986, IC2 LTR-303ALS-01, IC3 EFM32TG108F32, J1 Conn_01x05_Male, J2 Conn_01x04_Female, SW1 SW_Push

Commit message: More layout
Connections:
- IC3 pad 5: DPIN5 -> DPIN4
- IC3 pad 6: DPIN6 -> DPIN5
Routing:
- net DPIN4: track 117.8 -> 143.1 mm, vias 8 -> 12
- net DPIN5: track 117.1 -> 131.6 mm, vias 15 -> 17
- net GND: track 60.0 -> 57.3 mm
- net S3: track 109.4 -> 111.5 mm
- net DPIN6: track 157.2 -> 158.5 mm
- net RESET: track 32.8 -> 31.8 mm
- net DPIN1: track 152.1 -> 151.5 mm

Commit message: wiring complete
Connections:
- IC3 pad 17: S4 -> S2
- IC3 pad 18: S2 -> S4
Routing:
- net S2: track 14.1 -> 134.7 mm, vias 0 -> 3
- net S4: track 20.3 -> 105.4 mm, vias 0 -> 2
- net SWDIO: track 23.0 -> 24.3 mm
