File: board/board.kicad_pcb (KiCad board)
At the start: 2 copper layers, 50 x 81 mm, 79 parts, among them IC1 tps610981dser, IC2 LTR-303ALS-01, IC3 EFM32TG108F32, IC4 AT30TS74-SS8M-B, J1 Conn_01x05_Male, J2 , J3 , J4 , Q1 Q_PMOS_GSD, SW2 SW_SPST

Commit message: minor board tweaks
Routing:
- net DPIN6: track 201.1 -> 202.6 mm
- net DPIN5: track 122.2 -> 122.9 mm

Commit message: TEMP
Parts:
- added U1: TPL5010, Package_TO_SOT_SMD:SOT-23-6, F.Cu at (93.0, 57.7)
Connections:
- IC3 pad 10: REGMODE -> Net-(IC3-Pad10)
- IC3 pad 21: Net-(IC3-Pad21) -> REGMODE
Routing:
- net DPIN2: track 166.8 -> 172.7 mm
- net REGMODE: track 83.4 -> 88.8 mm
- net DPIN1: track 134.5 -> 137.6 mm
- net DPIN3: track 156.4 -> 158.6 mm
- net DPIN5: track 122.9 -> 124.9 mm
- net DPIN4: track 170.5 -> 172.1 mm
- net VBAT: track 61.9 -> 60.7 mm
- net AVREG: track 16.2 -> 15.6 mm

Commit message: TEMP BOARD MESS
Parts:
- removed D27: D_Schottky, Diode_SMD:D_SOD-523
- removed SW2: SW_SPST, mlm:CSS-1210TB
- moved U1 21.5 mm to (102.1, 77.2)
- moved C8 0.52 mm to (99.5, 74.1)
- moved C11 0.36 mm to (101.6, 74.1)
- moved R6 0.36 mm to (98.0, 74.1)
Connections:
- IC3 pad 10: Net-(IC3-Pad10) -> TPLDONE
- IC3 pad 11: Net-(IC3-Pad11) -> TPLWAKE
- U1 pad 4: Net-(U1-Pad4) -> TPLDONE
- U1 pad 5: Net-(U1-Pad5) -> TPLWAKE
Routing:
- net DPIN2: track 172.7 -> 151.3 mm
- net DPIN4: track 172.1 -> 151.1 mm, vias 10 -> 8
- net Net-(D27-Pad1): track 15.5 -> 0.00 mm
- net DPIN1: track 137.6 -> 125.7 mm
- net TPLDONE: track 0.00 -> 8.60 mm
- net TPLWAKE: track 0.00 -> 7.48 mm
- net Net-(IC3-Pad8): track 2.36 -> 0.62 mm
- net GND: track 204.5 -> 203.6 mm, vias 58 -> 57
- net Net-(IC3-Pad11): track 0.58 -> 0.00 mm

Commit message: TEMP
Parts:
- turned U1 to 180 degrees
Routing:
- net TPLDONE: track 8.60 -> 5.03 mm
- net PVREG: track 121.5 -> 119.4 mm
- net AVREG: track 15.6 -> 17.4 mm
- net DPIN2: track 151.3 -> 150.7 mm, vias 8 -> 6
- net DPIN3: track 158.6 -> 158.4 mm, vias 11 -> 9

Commit message: TEMP
Parts:
- moved L2 4.72 mm to (115.7, 76.7)
- moved R15 0.30 mm to (109.2, 73.3)
Routing:
- net VREG: track 126.1 -> 141.9 mm, vias 4 -> 6
- net Net-(L2-Pad2): track 13.1 -> 6.42 mm
- net DPIN1: track 125.7 -> 119.8 mm
- net Net-(IC3-Pad8): track 0.62 -> 2.27 mm
Other:
- rule trace_min: 0.18 -> 0.14

Commit message: board tweaks for next version
Parts:
- removed D25, D26: LED, mlm:dual0402
- moved MH5 16.2 mm to (79.3, 80.5)
- moved IC4 5.96 mm to (86.4, 79.1)
- moved D31 0.39 mm to (111.5, 77.3), turned to 180 degrees
- moved R5 0.07 mm to (88.5, 69.4)
Routing:
- net DPIN2: track 150.7 -> 141.9 mm, vias 6 -> 4
- net SCL: track 34.5 -> 41.1 mm
- net SDA: track 43.8 -> 49.4 mm, vias 0 -> 2
- net DPIN6: track 202.8 -> 197.5 mm, vias 13 -> 11
- net PVREG: track 119.4 -> 115.4 mm
- net VREG: track 141.9 -> 144.3 mm
- net GND: track 203.8 -> 202.5 mm, vias 57 -> 61

Commit message: board tweaks
Parts:
- added C15: u1, mlm:0603, F.Cu at (104.9, 77.0)
Routing:
- net GND: track 202.5 -> 204.4 mm, vias 61 -> 62
- net VREG: track 144.3 -> 145.7 mm
- net REGMODE: track 88.8 -> 89.9 mm, vias 4 -> 2
- net DPIN3: track 158.4 -> 159.6 mm
- net VBAT: track 60.7 -> 61.8 mm
- net Net-(C2-Pad1): track 1.02 -> 1.93 mm
- net DPIN1: track 119.5 -> 118.7 mm
- net DPIN2: track 141.9 -> 141.3 mm
