File: board/board.kicad_sch (KiCad schematic)
At the start: 95 parts, among them IC1 tps610981dser, IC2 LTR-303ALS-01, IC3 EFM32TG108F32-D-QFN24, IC4 AT30TS74-SS8M-B, IC5 ADA4528-2, IC6 TLV70245_SOT23-5, J1 Conn_01x05_Male, J2 , J3 , J4 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

Commit message: various mpn and value changes
Parts:
- D1, D10, D11, D12, D13, D14, D15, D16, D17, D18, D19, D2, D20, D21, D22, D23, D24, D3, D4, D5, D6, D7, D8, D9: MPN VLMB1500-GS08 -> IN-S42BT5B
- IC5: MPN ADA4528-2 -> ADA4528-2ACPZ-R7
- IC6: MPN TLV70245 -> TLV70245DBVT
- R10, R3, R4, R9: value 9.1 -> 23.2; MPN CRCW06039R10FKEA -> ERJ-2RKF23R2X
- R5: value 27 -> 23.2; MPN RMCF0603FT27R0 -> ERJ-2RKF23R2X

Commit message: fix wrong mpn
Parts:
- R6: value 9.1 -> 23.2; MPN CRCW06039R10FKEA -> ERJ-2RKF23R2X
Changed lines of the file:
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@@
 (kicad_sch (version 20200506) (host eeschema "(5.99.0-1555-g464399a0c)")
   (page "A0")
+  (junction (at 213.36 31.75))
+  (junction (at 82.55 53.34))
+  (junction (at 69.85 66.04))
+  (junction (at 200.66 31.75))
+  (junction (at 251.46 104.14))
+  (junction (at 53.34 167.64))
+  (junction (at 95.25 78.74))
+  (junction (at 48.26 38.1))
+  (junction (at 38.1 167.64))
+  (junction (at 401.32 49.53))
+  (junction (at 35.56 38.1))
+  (junction (at 31.75 40.64))
+  (junction (at 73.66 76.2))
+  (junction (at 360.68 96.52))
+  (junction (at 99.06 76.2))
+  (junction (at 86.36 25.4))
+  (junction (at 57.15 66.04))
+  (junction (at 374.65 49.53))
+  (junction (at 123.19 93.98))
+  (junction (at 35.56 50.8))
+  (junction (at 200.66 43.18))
+  (junction (at 372.11 49.53))
+  (junction (at 82.55 148.59))
+  (junction (at 82.55 38.1))
+  (junction (at 60.96 76.2))
+  (junction (at 48.26 63.5))
+  (junction (at 48.26 88.9))
+  (junction (at 57.15 40.64))
+  (junction (at 57.15 27.94))
+  (junction (at 213.36 21.59))
+  (junction (at 69.85 27.94))
+  (junction (at 82.55 66.04))
+  (junction (at 95.25 66.04))
+  (junction (at 187.96 53.34))
+  (junction (at 95.25 25.4))
+  (junction (at 219.71 93.98))
+  (junction (at 57.15 78.74))
+  (junction (at 60.96 88.9))
+  (junction (at 48.26 50.8))
+  (junction (at 44.45 76.2))
+  (junction (at 69.85 78.74))
+  (junction (at 48.26 25.4))
+  (junction (at 99.06 88.9))
+  (junction (at 116.84 153.67))
+  (junction (at 360.68 111.76))
+  (junction (at 31.75 27.94))
+  (junction (at 73.66 25.4))
+  (junction (at 44.45 27.94))
+  (junction (at 73.66 88.9))
+  (junction (at 31.75 53.34))
+  (junction (at 60.96 50.8))
+  (junction (at 44.45 78.74))
+  (junction (at 203.2 140.97))
+  (junction (at 24.13 167.64))
+  (junction (at 35.56 25.4))
+  (junction (at 60.96 38.1))
+  (junction (at 57.15 63.5))
+  (junction (at 73.66 38.1))
+  (junction (at 35.56 63.5))
+  (junction (at 342.9 99.06))
   (junction (at 139.7 93.98))
   (junction (at 378.46 96.52))
+  (junction (at 60.96 25.4))
+  (junction (at 345.44 93.98))
+  (junction (at 82.55 40.64))
+  (junction (at 86.36 76.2))
   (junction (at 86.36 50.8))
-  (junction (at 213.36 21.59))
-  (junction (at 203.2 154.94))
-  (junction (at 48.26 50.8))
-  (junction (at 82.55 148.59))
-  (junction (at 31.75 40.64))
-  (junction (at 57.15 63.5))
-  (junction (at 200.66 43.18))
-  (junction (at 73.66 63.5))
-  (junction (at 360.68 96.52))
-  (junction (at 95.25 66.04))
-  (junction (at 342.9 114.3))
+  (junction (at 203.2 31.75))
   (junction (at 31.75 88.9))
-  (junction (at 203.2 31.75))
-  (junction (at 57.15 78.74))
-  (junction (at 35.56 38.1))
-  (junction (at 82.55 53.34))
-  (junction (at 203.2 140.97))
-  (junction (at 69.85 53.34))
-  (junction (at 48.26 25.4))
-  (junction (at 116.84 99.06))
   (junction (at 44.45 40.64))
+  (junction (at 129.54 102.87))
+  (junction (at 187.96 154.94))
+  (junction (at 35.56 76.2))
+  (junction (at 31.75 66.04))
+  (junction (at 38.1 185.42))
   (junction (at 93.98 119.38))
-  (junction (at 48.26 63.5))
+  (junction (at 24.13 143.51))
+  (junction (at 69.85 166.37))
+  (junction (at 93.98 123.19))
+  (junction (at 364.49 83.82))
   (junction (at 69.85 50.8))
   (junction (at 334.01 86.36))
-  (junction (at 44.45 76.2))
-  (junction (at 60.96 76.2))
-  (junction (at 60.96 50.8))
-  (junction (at 24.13 167.64))
-  (junction (at 99.06 76.2))
-  (junction (at 73.66 76.2))
-  (junction (at 24.13 143.51))
-  (junction (at 48.26 38.1))
-  (junction (at 60.96 25.4))
-  (junction (at 69.85 78.74))
-  (junction (at 38.1 185.42))
-  (junction (at 35.56 76.2))
-  (junction (at 187.96 53.34))
-  (junction (at 35.56 25.4))
-  (junction (at 123.19 93.98))
-  (junction (at 38.1 167.64))
-  (junction (at 31.75 66.04))
-  (junction (at 82.55 66.04))
-  (junction (at 251.46 104.14))
-  (junction (at 82.55 40.64))
-  (junction (at 99.06 88.9))
-  (junction (at 372.11 49.53))
-  (junction (at 73.66 88.9))
-  (junction (at 364.49 83.82))
-  (junction (at 44.45 78.74))
-  (junction (at 82.55 38.1))
-  (junction (at 57.15 66.04))
-  (junction (at 57.15 40.64))
-  (junction (at 200.66 31.75))
-  (junction (at 60.96 88.9))
-  (junction (at 69.85 66.04))
-  (junction (at 360.68 111.76))
+  (junction (at 73.66 63.5))
   (junction (at 237.49 104.14))
-  (junction (at 95.25 25.4))
-  (junction (at 95.25 78.74))
-  (junction (at 116.84 153.67))
-  (junction (at 213.36 31.75))
-  (junction (at 35.56 63.5))
+  (junction (at 44.45 53.34))
   (junction (at 86.36 63.5))
-  (junction (at 31.75 27.94))
-  (junction (at 48.26 88.9))
-  (junction (at 219.71 93.98))
-  (junction (at 73.66 38.1))
-  (junction (at 401.32 49.53))
-  (junction (at 35.56 50.8))
-  (junction (at 53.34 167.64))
-  (junction (at 86.36 25.4))
-  (junction (at 73.66 25.4))
-  (junction (at 69.85 166.37))
-  (junction (at 60.96 38.1))
-  (junction (at 31.75 53.34))
-  (junction (at 345.44 93.98))
-  (junction (at 44.45 53.34))
-  (junction (at 342.9 99.06))
-  (junction (at 69.85 27.94))
-  (junction (at 374.65 49.53))
-  (junction (at 187.96 154.94))
-  (junction (at 44.45 27.94))
-  (junction (at 93.98 123.19))
-  (junction (at 129.54 102.87))
-  (junction (at 86.36 76.2))
-  (junction (at 57.15 27.94))
+  (junction (at 69.85 53.34))
+  (junction (at 342.9 114.3))
+  (junction (at 116.84 99.06))
+  (junction (at 203.2 154.94))
+  (no_connect (at 41.91 217.17))
+  (no_connect (at 27.94 217.17))
+  (no_connect (at 35.56 234.95))
+  (no_connect (at 72.39 119.38))
+  (no_connect (at 27.94 227.33))
+  (no_connect (at 193.04 129.54))
   (no_connect (at 198.12 129.54))
-  (no_connect (at 35.56 234.95))
-  (no_connect (at 193.04 129.54))
-  (no_connect (at 27.94 217.17))
   (no_connect (at 41.91 227.33))
   (no_connect (at 138.43 158.75))
-  (no_connect (at 27.94 227.33))
-  (no_connect (at 41.91 217.17))
-  (no_connect (at 72.39 119.38))
   (wire (pts (xy 19.05 167.64) (xy 24.13 167.64)))
   (wire (pts (xy 24.13 128.27) (xy 24.13 125.73)))
@@
   (symbol (lib_name "Device:R_9") (lib_id "Device:R") (at 182.88 135.89 180) (unit 1)
     (property "Reference" "R6" (id 0) (at 188.1378 135.89 90))
-    (property "Value" "9.1" (id 1) (at 185.8264 135.89 90))
+    (property "Value" "23.2" (id 1) (at 185.8264 135.89 90))
     (property "Footprint" "mlm:0603" (id 2) (at 184.658 135.89 90)
       (effects (font (size 1.27 1.27)) hide)
@@
       (effects (font (size 1.27 1.27)) hide)
     )
-    (property "MPN" "CRCW06039R10FKEA" (id 4) (at 396.24 91.44 0)
-      (effects (font (size 1.27 1.27)) hide)
-    )
+    (property "MPN" "ERJ-2RKF23R2X" (id 4) (at 396.24 91.44 0)
+      (effects (font (size 1.27 1.27)) hide)
+    )

Commit message: fix wrong mpns
Parts:
- R13: MPN RMCF0603FG1K00 -> RC0603FR-07100RL
Changed lines of the file:
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@@
 (kicad_sch (version 20200506) (host eeschema "(5.99.0-1555-g464399a0c)")
   (page "A0")
-  (junction (at 213.36 31.75))
+  (junction (at 31.75 88.9))
+  (junction (at 116.84 153.67))
+  (junction (at 95.25 25.4))
+  (junction (at 401.32 49.53))
+  (junction (at 82.55 40.64))
+  (junction (at 60.96 38.1))
+  (junction (at 31.75 53.34))
+  (junction (at 35.56 63.5))
+  (junction (at 342.9 99.06))
+  (junction (at 86.36 50.8))
+  (junction (at 237.49 104.14))
+  (junction (at 93.98 123.19))
+  (junction (at 57.15 66.04))
+  (junction (at 99.06 76.2))
+  (junction (at 364.49 83.82))
+  (junction (at 60.96 25.4))
+  (junction (at 69.85 78.74))
+  (junction (at 69.85 66.04))
+  (junction (at 57.15 78.74))
+  (junction (at 24.13 143.51))
+  (junction (at 48.26 50.8))
   (junction (at 82.55 53.34))
-  (junction (at 69.85 66.04))
-  (junction (at 200.66 31.75))
-  (junction (at 251.46 104.14))
-  (junction (at 53.34 167.64))
-  (junction (at 95.25 78.74))
-  (junction (at 48.26 38.1))
+  (junction (at 69.85 166.37))
+  (junction (at 129.54 102.87))
+  (junction (at 86.36 63.5))
+  (junction (at 95.25 66.04))
+  (junction (at 38.1 185.42))
+  (junction (at 73.66 38.1))
   (junction (at 38.1 167.64))
-  (junction (at 401.32 49.53))
-  (junction (at 35.56 38.1))
+  (junction (at 69.85 53.34))
   (junction (at 31.75 40.64))
-  (junction (at 73.66 76.2))
-  (junction (at 360.68 96.52))
-  (junction (at 99.06 76.2))
-  (junction (at 86.36 25.4))
-  (junction (at 57.15 66.04))
-  (junction (at 374.65 49.53))
-  (junction (at 123.19 93.98))
-  (junction (at 35.56 50.8))
-  (junction (at 200.66 43.18))
-  (junction (at 372.11 49.53))
-  (junction (at 82.55 148.59))
+  (junction (at 73.66 25.4))
+  (junction (at 44.45 76.2))
   (junction (at 82.55 38.1))
-  (junction (at 60.96 76.2))
-  (junction (at 48.26 63.5))
-  (junction (at 48.26 88.9))
-  (junction (at 57.15 40.64))
-  (junction (at 57.15 27.94))
   (junction (at 213.36 21.59))
   (junction (at 69.85 27.94))
-  (junction (at 82.55 66.04))
-  (junction (at 95.25 66.04))
-  (junction (at 187.96 53.34))
-  (junction (at 95.25 25.4))
-  (junction (at 219.71 93.98))
-  (junction (at 57.15 78.74))
   (junction (at 60.96 88.9))
-  (junction (at 48.26 50.8))
-  (junction (at 44.45 76.2))
-  (junction (at 69.85 78.74))
-  (junction (at 48.26 25.4))
-  (junction (at 99.06 88.9))
-  (junction (at 116.84 153.67))
-  (junction (at 360.68 111.76))
-  (junction (at 31.75 27.94))
-  (junction (at 73.66 25.4))
-  (junction (at 44.45 27.94))
-  (junction (at 73.66 88.9))
-  (junction (at 31.75 53.34))
-  (junction (at 60.96 50.8))
-  (junction (at 44.45 78.74))
-  (junction (at 203.2 140.97))
-  (junction (at 24.13 167.64))
-  (junction (at 35.56 25.4))
-  (junction (at 60.96 38.1))
   (junction (at 57.15 63.5))
-  (junction (at 73.66 38.1))
-  (junction (at 35.56 63.5))
-  (junction (at 342.9 99.06))
-  (junction (at 139.7 93.98))
-  (junction (at 378.46 96.52))
-  (junction (at 60.96 25.4))
-  (junction (at 345.44 93.98))
-  (junction (at 82.55 40.64))
-  (junction (at 86.36 76.2))
-  (junction (at 86.36 50.8))
-  (junction (at 203.2 31.75))
-  (junction (at 31.75 88.9))
-  (junction (at 44.45 40.64))
-  (junction (at 129.54 102.87))
-  (junction (at 187.96 154.94))
-  (junction (at 35.56 76.2))
-  (junction (at 31.75 66.04))
-  (junction (at 38.1 185.42))
-  (junction (at 93.98 119.38))
-  (junction (at 24.13 143.51))
-  (junction (at 69.85 166.37))
-  (junction (at 93.98 123.19))
-  (junction (at 364.49 83.82))
-  (junction (at 69.85 50.8))
-  (junction (at 334.01 86.36))
-  (junction (at 73.66 63.5))
-  (junction (at 237.49 104.14))
-  (junction (at 44.45 53.34))
-  (junction (at 86.36 63.5))
-  (junction (at 69.85 53.34))
-  (junction (at 342.9 114.3))
+  (junction (at 48.26 88.9))
   (junction (at 116.84 99.06))
   (junction (at 203.2 154.94))
+  (junction (at 44.45 40.64))
+  (junction (at 187.96 53.34))
+  (junction (at 57.15 40.64))
+  (junction (at 334.01 86.36))
+  (junction (at 139.7 93.98))
+  (junction (at 44.45 27.94))
+  (junction (at 69.85 50.8))
+  (junction (at 48.26 25.4))
+  (junction (at 372.11 49.53))
+  (junction (at 86.36 25.4))
+  (junction (at 200.66 43.18))
+  (junction (at 48.26 63.5))
+  (junction (at 219.71 93.98))
+  (junction (at 345.44 93.98))
+  (junction (at 48.26 38.1))
+  (junction (at 374.65 49.53))
+  (junction (at 73.66 63.5))
+  (junction (at 35.56 76.2))
+  (junction (at 187.96 154.94))
+  (junction (at 31.75 66.04))
+  (junction (at 360.68 96.52))
+  (junction (at 200.66 31.75))
+  (junction (at 95.25 78.74))
+  (junction (at 44.45 78.74))
+  (junction (at 35.56 25.4))
+  (junction (at 60.96 76.2))
+  (junction (at 99.06 88.9))
+  (junction (at 35.56 50.8))
+  (junction (at 24.13 167.64))
+  (junction (at 203.2 140.97))
+  (junction (at 93.98 119.38))
+  (junction (at 31.75 27.94))
+  (junction (at 82.55 148.59))
+  (junction (at 35.56 38.1))
+  (junction (at 73.66 88.9))
+  (junction (at 123.19 93.98))
+  (junction (at 53.34 167.64))
+  (junction (at 60.96 50.8))
+  (junction (at 251.46 104.14))
+  (junction (at 378.46 96.52))
+  (junction (at 44.45 53.34))
+  (junction (at 342.9 114.3))
+  (junction (at 82.55 66.04))
+  (junction (at 213.36 31.75))
+  (junction (at 203.2 31.75))
+  (junction (at 73.66 76.2))
+  (junction (at 57.15 27.94))
+  (junction (at 86.36 76.2))
+  (junction (at 360.68 111.76))
+  (no_connect (at 193.04 129.54))
+  (no_connect (at 27.94 217.17))
+  (no_connect (at 138.43 158.75))
+  (no_connect (at 198.12 129.54))
+  (no_connect (at 27.94 227.33))
+  (no_connect (at 72.39 119.38))
   (no_connect (at 41.91 217.17))
-  (no_connect (at 27.94 217.17))
   (no_connect (at 35.56 234.95))
-  (no_connect (at 72.39 119.38))
-  (no_connect (at 27.94 227.33))
-  (no_connect (at 193.04 129.54))
-  (no_connect (at 198.12 129.54))
   (no_connect (at 41.91 227.33))
-  (no_connect (at 138.43 158.75))
   (wire (pts (xy 19.05 167.64) (xy 24.13 167.64)))
   (wire (pts (xy 24.13 128.27) (xy 24.13 125.73)))
@@
     )
   )
-  (symbol (lib_id "Device:R") (at 116.84 109.22 180) (unit 1)
+  (symbol (lib_name "Device:R_13") (lib_id "Device:R") (at 116.84 109.22 180) (unit 1)
     (property "Reference" "R13" (id 0) (at 122.0978 109.22 90))
     (property "Value" "100" (id 1) (at 119.7864 109.22 90))
@@
       (effects (font (size 1.27 1.27)) hide)
     )
-    (property "MPN" "RMCF0603FG1K00" (id 4) (at 330.2 55.88 0)
+    (property "MPN" "RC0603FR-07100RL" (id 4) (at 330.2 55.88 0)
       (effects (font (size 1.27 1.27)) hide)
     )
@@
     )
   )
-  (symbol (lib_id "Device:R") (at 229.87 93.98 270) (unit 1)
+  (symbol (lib_name "Device:R_14") (lib_id "Device:R") (at 229.87 93.98 270) (unit 1)
     (property "Reference" "R15" (id 0) (at 229.87 88.7222 90))
     (property "Value" "100" (id 1) (at 229.87 91.0336 90))

Commit message: sync board and sch
Parts:
- C17: MPN GRM188R60J106ME84D -> 885012206020
- D25, D26: MPN (none) -> IN-S42BT5B
Changed lines of the file:
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@@
 (kicad_sch (version 20200506) (host eeschema "(5.99.0-1555-g464399a0c)")
   (page "A0")
+  (junction (at 342.9 99.06))
+  (junction (at 60.96 76.2))
+  (junction (at 48.26 88.9))
+  (junction (at 48.26 38.1))
+  (junction (at 82.55 53.34))
+  (junction (at 69.85 27.94))
+  (junction (at 35.56 25.4))
+  (junction (at 35.56 76.2))
+  (junction (at 82.55 66.04))
+  (junction (at 82.55 148.59))
+  (junction (at 95.25 78.74))
+  (junction (at 24.13 167.64))
+  (junction (at 44.45 27.94))
+  (junction (at 60.96 25.4))
+  (junction (at 187.96 53.34))
+  (junction (at 69.85 50.8))
+  (junction (at 86.36 50.8))
+  (junction (at 93.98 123.19))
+  (junction (at 116.84 99.06))
+  (junction (at 378.46 96.52))
+  (junction (at 69.85 78.74))
+  (junction (at 401.32 49.53))
+  (junction (at 44.45 53.34))
+  (junction (at 44.45 40.64))
+  (junction (at 35.56 38.1))
+  (junction (at 73.66 76.2))
+  (junction (at 364.49 83.82))
+  (junction (at 374.65 49.53))
+  (junction (at 203.2 31.75))
+  (junction (at 35.56 63.5))
+  (junction (at 116.84 153.67))
+  (junction (at 82.55 38.1))
+  (junction (at 60.96 88.9))
+  (junction (at 60.96 50.8))
+  (junction (at 95.25 25.4))
+  (junction (at 31.75 66.04))
+  (junction (at 139.7 93.98))
+  (junction (at 237.49 104.14))
+  (junction (at 219.71 93.98))
+  (junction (at 57.15 27.94))
+  (junction (at 57.15 40.64))
+  (junction (at 372.11 49.53))
+  (junction (at 203.2 154.94))
+  (junction (at 360.68 111.76))
+  (junction (at 38.1 185.42))
+  (junction (at 95.25 66.04))
+  (junction (at 200.66 31.75))
+  (junction (at 38.1 167.64))
+  (junction (at 123.19 93.98))
+  (junction (at 73.66 25.4))
+  (junction (at 69.85 66.04))
+  (junction (at 203.2 140.97))
   (junction (at 31.75 88.9))
-  (junction (at 116.84 153.67))
-  (junction (at 95.25 25.4))
-  (junction (at 401.32 49.53))
+  (junction (at 73.66 88.9))
+  (junction (at 73.66 63.5))
+  (junction (at 31.75 40.64))
+  (junction (at 334.01 86.36))
+  (junction (at 86.36 63.5))
+  (junction (at 360.68 96.52))
+  (junction (at 48.26 50.8))
+  (junction (at 31.75 27.94))
+  (junction (at 342.9 114.3))
+  (junction (at 31.75 53.34))
+  (junction (at 48.26 25.4))
+  (junction (at 200.66 43.18))
+  (junction (at 57.15 63.5))
+  (junction (at 213.36 21.59))
+  (junction (at 69.85 53.34))
   (junction (at 82.55 40.64))
   (junction (at 60.96 38.1))
-  (junction (at 31.75 53.34))
-  (junction (at 35.56 63.5))
-  (junction (at 342.9 99.06))
-  (junction (at 86.36 50.8))
-  (junction (at 237.49 104.14))
-  (junction (at 93.98 123.19))
+  (junction (at 73.66 38.1))
+  (junction (at 24.13 143.51))
+  (junction (at 99.06 76.2))
   (junction (at 57.15 66.04))
-  (junction (at 99.06 76.2))
-  (junction (at 364.49 83.82))
-  (junction (at 60.96 25.4))
-  (junction (at 69.85 78.74))
-  (junction (at 69.85 66.04))
+  (junction (at 69.85 166.37))
+  (junction (at 187.96 154.94))
   (junction (at 57.15 78.74))
-  (junction (at 24.13 143.51))
-  (junction (at 48.26 50.8))
-  (junction (at 82.55 53.34))
-  (junction (at 69.85 166.37))
   (junction (at 129.54 102.87))
-  (junction (at 86.36 63.5))
-  (junction (at 95.25 66.04))
-  (junction (at 38.1 185.42))
-  (junction (at 73.66 38.1))
-  (junction (at 38.1 167.64))
-  (junction (at 69.85 53.34))
-  (junction (at 31.75 40.64))
-  (junction (at 73.66 25.4))
+  (junction (at 35.56 50.8))
+  (junction (at 86.36 25.4))
+  (junction (at 99.06 88.9))
+  (junction (at 44.45 78.74))
+  (junction (at 213.36 31.75))
+  (junction (at 53.34 167.64))
+  (junction (at 345.44 93.98))
+  (junction (at 251.46 104.14))
+  (junction (at 48.26 63.5))
+  (junction (at 86.36 76.2))
+  (junction (at 93.98 119.38))
   (junction (at 44.45 76.2))
-  (junction (at 82.55 38.1))
-  (junction (at 213.36 21.59))
-  (junction (at 69.85 27.94))
-  (junction (at 60.96 88.9))
-  (junction (at 57.15 63.5))
-  (junction (at 48.26 88.9))
-  (junction (at 116.84 99.06))
-  (junction (at 203.2 154.94))
-  (junction (at 44.45 40.64))
-  (junction (at 187.96 53.34))
-  (junction (at 57.15 40.64))
-  (junction (at 334.01 86.36))
-  (junction (at 139.7 93.98))
-  (junction (at 44.45 27.94))
-  (junction (at 69.85 50.8))
-  (junction (at 48.26 25.4))
-  (junction (at 372.11 49.53))
-  (junction (at 86.36 25.4))
-  (junction (at 200.66 43.18))
-  (junction (at 48.26 63.5))
-  (junction (at 219.71 93.98))
-  (junction (at 345.44 93.98))
-  (junction (at 48.26 38.1))
-  (junction (at 374.65 49.53))
-  (junction (at 73.66 63.5))
-  (junction (at 35.56 76.2))
-  (junction (at 187.96 154.94))
-  (junction (at 31.75 66.04))
-  (junction (at 360.68 96.52))
-  (junction (at 200.66 31.75))
-  (junction (at 95.25 78.74))
-  (junction (at 44.45 78.74))
-  (junction (at 35.56 25.4))
-  (junction (at 60.96 76.2))
-  (junction (at 99.06 88.9))
-  (junction (at 35.56 50.8))
-  (junction (at 24.13 167.64))
-  (junction (at 203.2 140.97))
-  (junction (at 93.98 119.38))
-  (junction (at 31.75 27.94))
-  (junction (at 82.55 148.59))
-  (junction (at 35.56 38.1))
-  (junction (at 73.66 88.9))
-  (junction (at 123.19 93.98))
-  (junction (at 53.34 167.64))
-  (junction (at 60.96 50.8))
-  (junction (at 251.46 104.14))
-  (junction (at 378.46 96.52))
-  (junction (at 44.45 53.34))
-  (junction (at 342.9 114.3))
-  (junction (at 82.55 66.04))
-  (junction (at 213.36 31.75))
-  (junction (at 203.2 31.75))
-  (junction (at 73.66 76.2))
-  (junction (at 57.15 27.94))
-  (junction (at 86.36 76.2))
-  (junction (at 360.68 111.76))
+  (no_connect (at 72.39 119.38))
+  (no_connect (at 198.12 129.54))
+  (no_connect (at 41.91 227.33))
+  (no_connect (at 41.91 217.17))
   (no_connect (at 193.04 129.54))
+  (no_connect (at 35.56 234.95))
   (no_connect (at 27.94 217.17))
   (no_connect (at 138.43 158.75))
-  (no_connect (at 198.12 129.54))
   (no_connect (at 27.94 227.33))
-  (no_connect (at 72.39 119.38))
-  (no_connect (at 41.91 217.17))
-  (no_connect (at 35.56 234.95))
-  (no_connect (at 41.91 227.33))
   (wire (pts (xy 19.05 167.64) (xy 24.13 167.64)))
   (wire (pts (xy 24.13 128.27) (xy 24.13 125.73)))
@@
     )
   )
-  (symbol (lib_id "Device:LED_ALT") (at 99.06 69.85 90) (unit 1)
+  (symbol (lib_name "Device:LED_ALT_1") (lib_id "Device:LED_ALT") (at 99.06 69.85 90) (unit 1)
     (property "Reference" "D25" (id 0) (at 102.0572 68.8594 90)
       (effects (font (size 1.27 1.27)) (justify right))
@@
     )
     (property "Datasheet" "~" (id 3) (at 99.06 69.85 0)
+      (effects (font (size 1.27 1.27)) hide)
+    )
+    (property "MPN" "IN-S42BT5B" (id 4) (at 99.06 69.85 90)
       (effects (font (size 1.27 1.27)) hide)
     )
@@
     )
     (property "Datasheet" "~" (id 3) (at 99.06 82.55 0)
+      (effects (font (size 1.27 1.27)) hide)
+    )
+    (property "MPN" "IN-S42BT5B" (id 4) (at 99.06 82.55 90)
       (effects (font (size 1.27 1.27)) hide)
     )
@@
     )
   )
-  (symbol (lib_id "pspice:CAP") (at 175.26 53.34 90) (unit 1)
+  (symbol (lib_name "pspice:CAP_4") (lib_id "pspice:CAP") (at 175.26 53.34 90) (unit 1)
     (property "Reference" "C9" (id 0) (at 175.26 45.339 90))
     (property "Value" "u1" (id 1) (at 175.26 47.6504 90))
@@
       (effects (font (size 1.27 1.27)) hide)
     )
-    (property "MPN" "GRM188R60J106ME84D" (id 4) (at 346.71 53.34 0)
-      (effects (font (size 1.27 1.27)) hide)
-    )
+    (property "MPN" "885012206020" (id 4) (at 346.71 53.34 0)
+      (effects (font (size 1.27 1.27)) hide)
+    )
