File: board/board.kicad_sch (KiCad schematic)
At the start: 81 parts, among them IC1 tps610981dser, IC2 LTR-303ALS-01, IC3 EFM32TG108F32-D-QFN24, J1 Conn_01x05_Male, J2 , J3 , J4 , Q1 Q_PMOS_GSD, Q2 Q_PMOS_GSD

Commit message: attempt to reduce total capacitance a little
Parts:
- added C19: 1u, mlm:0603, symbol pspice:CAP
- C1: footprint Capacitor_SMD:C_1206_3216Metric -> mlm:0603; MAN Kemet -> Samsung Electro-Mechanics; MPN C1206C475J3RACTU -> C0603C475K9PAC7411
- C10, C12: value 10u -> 4u7; MAN Taiyo Yuden -> Kemet; MPN JMK107ABJ106MA-T -> C0603C475K9PAC7411
Connections:
- net GND: now also C19.2
- net VREG: now also C19.1
Other:
- moved on the sheet: C1
Changed lines of the file:
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@@
   (junction (at 20.32 167.64) (diameter 1.016) (color 0 0 0 0))
   (junction (at 20.32 186.69) (diameter 1.016) (color 0 0 0 0))
-  (junction (at 24.13 143.51) (diameter 1.016) (color 0 0 0 0))
+  (junction (at 22.86 143.51) (diameter 1.016) (color 0 0 0 0))
   (junction (at 31.75 27.94) (diameter 1.016) (color 0 0 0 0))
   (junction (at 31.75 40.64) (diameter 1.016) (color 0 0 0 0))
@@
   (junction (at 35.56 63.5) (diameter 1.016) (color 0 0 0 0))
   (junction (at 35.56 76.2) (diameter 1.016) (color 0 0 0 0))
+  (junction (at 36.83 143.51) (diameter 1.016) (color 0 0 0 0))
   (junction (at 39.37 167.64) (diameter 1.016) (color 0 0 0 0))
   (junction (at 44.45 27.94) (diameter 1.016) (color 0 0 0 0))
@@
     (stroke (width 0) (type solid) (color 0 0 0 0))
   )
-  (wire (pts (xy 24.13 128.27) (xy 24.13 125.73))
+  (wire (pts (xy 22.86 128.27) (xy 22.86 125.73))
     (stroke (width 0) (type solid) (color 0 0 0 0))
   )
-  (wire (pts (xy 24.13 140.97) (xy 24.13 143.51))
+  (wire (pts (xy 22.86 140.97) (xy 22.86 143.51))
     (stroke (width 0) (type solid) (color 0 0 0 0))
   )
-  (wire (pts (xy 24.13 143.51) (xy 20.32 143.51))
+  (wire (pts (xy 22.86 143.51) (xy 20.32 143.51))
     (stroke (width 0) (type solid) (color 0 0 0 0))
   )
@@
     (stroke (width 0) (type solid) (color 0 0 0 0))
   )
+  (wire (pts (xy 36.83 125.73) (xy 36.83 128.27))
+    (stroke (width 0) (type solid) (color 0 0 0 0))
+  )
+  (wire (pts (xy 36.83 140.97) (xy 36.83 143.51))
+    (stroke (width 0) (type solid) (color 0 0 0 0))
+  )
+  (wire (pts (xy 36.83 143.51) (xy 22.86 143.51))
+    (stroke (width 0) (type solid) (color 0 0 0 0))
+  )
   (wire (pts (xy 39.37 153.67) (xy 39.37 167.64))
     (stroke (width 0) (type solid) (color 0 0 0 0))
@@
     (stroke (width 0) (type solid) (color 0 0 0 0))
   )
-  (wire (pts (xy 41.91 143.51) (xy 24.13 143.51))
+  (wire (pts (xy 41.91 143.51) (xy 36.83 143.51))
     (stroke (width 0) (type solid) (color 0 0 0 0))
   )
@@
     )
   )
-  (symbol (lib_id "power:GND") (at 24.13 125.73 180) (unit 1)
+  (symbol (lib_id "power:GND") (at 22.86 125.73 180) (unit 1)
+    (in_bom yes) (on_board yes)
+    (property "Reference" "#PWR01" (id 0) (at 22.86 119.38 0)
+      (effects (font (size 1.27 1.27)) hide)
+    )
+    (property "Value" "GND" (id 1) (at 22.733 122.4788 90)
+      (effects (font (size 1.27 1.27)) (justify right))
+    )
+    (property "Footprint" "" (id 2) (at 22.86 125.73 0)
+      (effects (font (size 1.27 1.27)) hide)
+    )
+    (property "Datasheet" "" (id 3) (at 22.86 125.73 0)
+      (effects (font (size 1.27 1.27)) hide)
+    )
+  )
+  (symbol (lib_id "power:GND") (at 36.83 125.73 180) (unit 1)
     (in_bom yes) (on_board yes)
-    (property "Reference" "#PWR01" (id 0) (at 24.13 119.38 0)
+    (property "Reference" "#PWR0101" (id 0) (at 36.83 119.38 0)
       (effects (font (size 1.27 1.27)) hide)
     )
-    (property "Value" "GND" (id 1) (at 24.003 122.4788 90)
+    (property "Value" "GND" (id 1) (at 36.703 122.4788 90)
       (effects (font (size 1.27 1.27)) (justify right))
     )
-    (property "Footprint" "" (id 2) (at 24.13 125.73 0)
+    (property "Footprint" "" (id 2) (at 36.83 125.73 0)
       (effects (font (size 1.27 1.27)) hide)
     )
-    (property "Datasheet" "" (id 3) (at 24.13 125.73 0)
+    (property "Datasheet" "" (id 3) (at 36.83 125.73 0)
       (effects (font (size 1.27 1.27)) hide)
     )
@@
     )
   )
-  (symbol (lib_name "pspice:CAP_7") (lib_id "pspice:CAP") (at 24.13 134.62 180) (unit 1)
+  (symbol (lib_name "pspice:CAP_7") (lib_id "pspice:CAP") (at 22.86 134.62 180) (unit 1)
     (in_bom yes) (on_board yes)
-    (property "Reference" "C1" (id 0) (at 32.131 134.62 90))
-    (property "Value" "4u7" (id 1) (at 29.8196 134.62 90))
-    (property "Footprint" "Capacitor_SMD:C_1206_3216Metric" (id 2) (at 24.13 134.62 0)
+    (property "Reference" "C1" (id 0) (at 30.861 134.62 90))
+    (property "Value" "4u7" (id 1) (at 28.5496 134.62 90))
+    (property "Footprint" "mlm:0603" (id 2) (at 22.86 134.62 0)
       (effects (font (size 1.27 1.27)) hide)
     )
-    (property "Datasheet" "~" (id 3) (at 24.13 134.62 0)
+    (property "Datasheet" "~" (id 3) (at 22.86 134.62 0)
       (effects (font (size 1.27 1.27)) hide)
     )
-    (property "MPN" "C1206C475J3RACTU" (id 4) (at 24.13 134.62 90)
+    (property "MPN" "C0603C475K9PAC7411" (id 4) (at 22.86 134.62 90)
       (effects (font (size 1.27 1.27)) hide)
     )
-    (property "MAN" "Kemet" (id 5) (at 24.13 134.62 90)
+    (property "MAN" "Samsung Electro-Mechanics" (id 5) (at 22.86 134.62 90)
       (effects (font (size 1.27 1.27)) hide)
     )
@@
     )
   )
+  (symbol (lib_name "pspice:CAP_6") (lib_id "pspice:CAP") (at 36.83 134.62 180) (unit 1)
+    (in_bom yes) (on_board yes)
+    (property "Reference" "C19" (id 0) (at 41.3512 133.4516 0)
+      (effects (font (size 1.27 1.27)) (justify right))
+    )
+    (property "Value" "1u" (id 1) (at 41.3512 135.763 0)
+      (effects (font (size 1.27 1.27)) (justify right))
+    )
+    (property "Footprint" "mlm:0603" (id 2) (at 36.83 134.62 0)
+      (effects (font (size 1.27 1.27)) hide)
+    )
+    (property "Datasheet" "~" (id 3) (at 36.83 134.62 0)
+      (effects (font (size 1.27 1.27)) hide)
+    )
+    (property "MPN" "CL10B105KP8NNNC" (id 4) (at 36.83 134.62 0)
+      (effects (font (size 1.27 1.27)) hide)
+    )
+    (property "MAN" "Wurth Elektronik" (id 5) (at 36.83 134.62 0)
+      (effects (font (size 1.27 1.27)) hide)
+    )
+  )
   (symbol (lib_name "pspice:CAP_11") (lib_id "pspice:CAP") (at 46.99 179.07 180) (unit 1)
     (in_bom yes) (on_board yes)
@@
     (in_bom yes) (on_board yes)
     (property "Reference" "C10" (id 0) (at 214.63 132.969 90))
-    (property "Value" "10u" (id 1) (at 214.63 135.2804 90))
+    (property "Value" "4u7" (id 1) (at 214.63 135.2804 90))
     (property "Footprint" "mlm:0603" (id 2) (at 214.63 140.97 0)
       (effects (font (size 1.27 1.27)) hide)
@@
       (effects (font (size 1.27 1.27)) hide)
     )
-    (property "MPN" "JMK107ABJ106MA-T" (id 4) (at 214.63 140.97 90)
+    (property "MPN" "C0603C475K9PAC7411" (id 4) (at 214.63 140.97 90)
       (effects (font (size 1.27 1.27)) hide)
     )
-    (property "MAN" "Taiyo Yuden" (id 5) (at 214.63 140.97 90)
+    (property "MAN" "Kemet" (id 5) (at 214.63 140.97 90)
       (effects (font (size 1.27 1.27)) hide)
     )
@@
       (effects (font (size 1.27 1.27)) (justify right))
     )
-    (property "Value" "10u" (id 1) (at 242.0112 121.793 0)
+    (property "Value" "4u7" (id 1) (at 242.0112 121.793 0)
       (effects (font (size 1.27 1.27)) (justify right))
     )
@@
       (effects (font (size 1.27 1.27)) hide)
     )
-    (property "MPN" "JMK107ABJ106MA-T" (id 4) (at 237.49 120.65 0)
+    (property "MPN" "C0603C475K9PAC7411" (id 4) (at 237.49 120.65 0)
       (effects (font (size 1.27 1.27)) hide)
     )
-    (property "MAN" "Taiyo Yuden" (id 5) (at 237.49 120.65 0)
+    (property "MAN" "Kemet" (id 5) (at 237.49 120.65 0)
       (effects (font (size 1.27 1.27)) hide)
     )
@@
       (reference "#PWR021") (unit 1) (value "GND") (footprint "")
     )
+    (path "/4acc0e38-5194-4381-b49c-ef38fde779ab"
+      (reference "#PWR0101") (unit 1) (value "GND") (footprint "")
+    )
     (path "/a04503d3-704e-464c-8cc1-3a97192a7e30"
       (reference "#PWR0102") (unit 1) (value "GND") (footprint "")
@@
     )
     (path "/cf55fafc-e904-492f-a59c-c6054a833ef5"
-      (reference "C1") (unit 1) (value "4u7") (footprint "Capacitor_SMD:C_1206_3216Metric")
+      (reference "C1") (unit 1) (value "4u7") (footprint "mlm:0603")
     )
     (path "/d342d333-a313-4d6a-9273-353c5c3efa8d"
@@
     )
     (path "/fd69a6a2-4a78-4260-9161-393990d4bb7e"
-      (reference "C10") (unit 1) (value "10u") (footprint "mlm:0603")
+      (reference "C10") (unit 1) (value "4u7") (footprint "mlm:0603")
     )
     (path "/3faa88c9-b29b-40df-a8d6-3af464413742"
@@
     )
     (path "/ec53c20d-8665-488b-98e4-bc1de125e602"
-      (reference "C12") (unit 1) (value "10u") (footprint "mlm:0603")
+      (reference "C12") (unit 1) (value "4u7") (footprint "mlm:0603")
     )
     (path "/b8a4f687-ccdb-42e5-b09d-f8beae72d8ef"
@@
       (reference "C18") (unit 1) (value "u1") (footprint "mlm:0603")
     )
+    (path "/265f1272-c35c-44b2-bc61-a449afef1ad3"
+      (reference "C19") (unit 1) (value "1u") (footprint "mlm:0603")
+    )
     (path "/069dfa89-be4b-478f-b58a-a1f91699b089"
